File: hardware/FTController.sch (KiCad schematic (older format))
At the start: 42 parts, among them IC1 ATMEGA328-AU, J1 RF, J2 RF_A, J3 RF_B, P1 9V IN, P10 LCD_BACKLIGHT, P2 COUNTER, P3 LCD, P4 AVR-ISP, U1 LD1117S33TR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

Commit message: Updated KiCAD files for KiCAD 5.0 and exported schematics
Parts:
- C1, C11, C4: symbol CP -> device:CP
- C10, C2, C3, C5, C6, C7, C8, C9: symbol C -> device:C
- D1, D3: symbol D -> device:D
- D2: symbol LED -> device:LED
- F1: symbol Polyfuse -> device:Polyfuse
- IC1: symbol ATMEGA328-AU -> FTController-rescue:ATMEGA328-AU
- J1, J2, J3, P1, P10, P2: symbol CONN_01X02 -> tinkerforge:CONN_01X02
- MK1, MK2, MK3, MK4: symbol Mounting_Hole -> FTController-rescue:Mounting_Hole
- P3: symbol CONN_02X05 -> FTController-rescue:CONN_02X05
- P4: symbol AVR-ISP -> avr-isp:AVR-ISP
- R1, R2, R24, R3, R4, R5: symbol R -> device:R
- RV1: symbol POT_TRIM -> FTController-rescue:POT_TRIM
- U1: symbol LD1117S33TR -> FTController-rescue:LD1117S33TR
- U2: symbol CNY17-1 -> FTController-rescue:CNY17-1
- U3: symbol LM78L05ACZ -> FTController-rescue:LM78L05ACZ
- U4, U5: symbol JOYSTICK_BUTTON -> tinkerforge:JOYSTICK_BUTTON
- U6: symbol NRF24L01 -> nrf24l01-connector:NRF24L01
- Y1: symbol Crystal -> device:Crystal
